File: kicad/keyboard2.kicad_pcb (KiCad board)
At the start: 2 copper layers, 317.5 x 103.2 mm, 181 parts, among them J1 Conn_02x06_Odd_Even, J2 Conn_01x12, J3 Conn_01x12_MountingPin, J4 USB_B_Mini, J5 Conn_02x03_Odd_Even, SW1 SW_Push, SW10 SW_Push, SW11 SW_Push, SW12 SW_Push, SW13 SW_Push, SW14 SW_Push, SW15 SW_Push, SW16 SW_Push, SW17 SW_Push, SW18 SW_Push, SW19 SW_Push, SW2 SW_Push, SW20 SW_Push, SW21 SW_Push, SW22 SW_Push, SW23 SW_Push, SW24 SW_Push, SW25 SW_Push, SW26 SW_Push, SW27 SW_Push, SW28 SW_Push, SW29 SW_Push, SW3 SW_Push, SW30 SW_Push, SW31 SW_Push, SW32 SW_Push, SW33 SW_Push, SW34 SW_Push, SW35 SW_Push, SW36 SW_Push, SW37 SW_Push, SW38 SW_Push, SW39 SW_Push, SW4 SW_Push, SW40 SW_Push, SW41 SW_Push, SW42 SW_Push, SW43 SW_Push, SW44 SW_Push, SW45 SW_Push, SW46 SW_Push, SW47 SW_Push, SW48 SW_Push, SW49 SW_Push, SW5 SW_Push, SW50 SW_Push, SW51 SW_Push, SW52 SW_Push, SW53 SW_Push, SW54 SW_Push, SW55 SW_Push, SW56 SW_Push, SW57 SW_Push, SW58 SW_Push, SW59 SW_Push, SW6 SW_Push, SW60 SW_Push, SW61 SW_Push, SW62 SW_Push, SW63 SW_Push, SW64 SW_Push, SW65 SW_Push, SW66 SW_Push, SW67 SW_Push, SW68 SW_Push, SW7 SW_Push, SW8 SW_Push, SW9 SW_Push, U1 74HC138, U2 74HC138, U3 ATmega16U4-A, Y1 Crystal

Commit message: Revision B:
- fix wrong space size (6.5u -> 6.25u),
- fix wrong right shift size (2u -> 1.75u),
- fix wrong placement of space stabilizer,
- fix J1 being mirrored against IDC-12 connector,
- change diodes footprint (hand soldering version has way too big pads),
- reroute.
Parts:
- removed the REF** at (198.4, 181.3)
- removed the REF** at (183.8, 180.7)
- removed the REF** at (360.5, 94.5)
- removed the REF** at (337.3, 142.8)
- removed the REF** at (92.1, 161.8)
- removed the REF** at (302.9, 161.7)
- removed the REF** at (360.5, 190.7)
- removed the REF** at (205.2, 190.7)
- removed the REF** at (319.6, 104.5)
- removed the REF** at (125.6, 186.0)
- removed the REF** at (50.0, 190.7)
- removed the REF** at (300.0, 104.4)
- removed the REF** at (216.8, 180.5)
- removed the REF** at (242.1, 186.0)
- removed the REF** at (76.0, 127.5)
- removed the REF** at (50.0, 142.6)
- removed the REF** at (71.9, 161.7)
- removed the REF** at (50.0, 94.5)
- removed the REF** at (317.2, 142.6)
- added REF**: MountingHole_3.2mm_M3_Pad_Via, MountingHole:MountingHole_3.2mm_M3_Pad_Via, F.Cu at (45.1, 61.3)
- added REF**: MountingHole_3.2mm_M3_Pad_Via, MountingHole:MountingHole_3.2mm_M3_Pad_Via, F.Cu at (45.1, 156.5)
- added REF**: MountingHole_3.2mm_M3_Pad_Via, MountingHole:MountingHole_3.2mm_M3_Pad_Via, F.Cu at (349.9, 156.5)
- added REF**: MountingHole_3.2mm_M3_Pad_Via, MountingHole:MountingHole_3.2mm_M3_Pad_Via, F.Cu at (349.9, 61.3)
- D1, D10, D11, D12, D13, D14, D15, D16, D17, D18, D19, D2, D20, D21, D22, D23, D24, D25, D26, D27, D28, D29, D3, D30, D31, D32, D33, D34, D35, D36, D37, D38, D39, D4, D40, D41, D42, D43, D44, D45, D46, D47, D48, D49, D5, D50, D51, D52, D53, D54, D55, D56, D57, D58, D59, D6, D60, D61, D62, D63, D64, D65, D66, D67, D68, D7, D8, D9: footprint Diode_SMD:D_MiniMELF_Handsoldering -> Diode_SMD:D_MiniMELF
- J1: footprint Connector_PinSocket_2.54mm:PinSocket_2x06_P2.54mm_Vertical -> Connector_IDC:IDC-Header_2x06_P2.54mm_Vertical
- SW1, SW10, SW11, SW12, SW13, SW15, SW17, SW18, SW19, SW2, SW20, SW21, SW22, SW23, SW24, SW25, SW26, SW27, SW28, SW3, SW30, SW32, SW33, SW34, SW35, SW36, SW37, SW38, SW39, SW4, SW40, SW41, SW42, SW44, SW46, SW47, SW48, SW49, SW5, SW50, SW51, SW52, SW53, SW54, SW55, SW57, SW58, SW6, SW63, SW64, SW65, SW66, SW67, SW68, SW7, SW8, SW9: footprint PCM_Switch_Keyboard_Cherry_MX:SW_Cherry_MX_PCB_1.00u -> Button_Switch_Keyboard:SW_Cherry_MX_1.00u_PCB
- SW14: footprint PCM_Switch_Keyboard_Cherry_MX:SW_Cherry_MX_PCB_2.25u -> Button_Switch_Keyboard:SW_Cherry_MX_2.00u_PCB
- SW16: footprint PCM_Switch_Keyboard_Cherry_MX:SW_Cherry_MX_PCB_1.50u -> Button_Switch_Keyboard:SW_Cherry_MX_1.50u_PCB
- SW29: footprint PCM_Switch_Keyboard_Cherry_MX:SW_Cherry_MX_PCB_1.75u -> Button_Switch_Keyboard:SW_Cherry_MX_1.50u_PCB
- SW31: footprint PCM_Switch_Keyboard_Cherry_MX:SW_Cherry_MX_PCB_1.75u -> Button_Switch_Keyboard:SW_Cherry_MX_1.75u_PCB
- SW43: footprint PCM_Switch_Keyboard_Cherry_MX:SW_Cherry_MX_PCB_2.50u -> Button_Switch_Keyboard:SW_Cherry_MX_2.25u_PCB
- SW45: footprint PCM_Switch_Keyboard_Cherry_MX:SW_Cherry_MX_PCB_2.25u -> Button_Switch_Keyboard:SW_Cherry_MX_2.25u_PCB
- SW56: footprint PCM_Switch_Keyboard_Cherry_MX:SW_Cherry_MX_PCB_2.00u -> Button_Switch_Keyboard:SW_Cherry_MX_1.75u_PCB
- SW59, SW60, SW61: footprint PCM_Switch_Keyboard_Cherry_MX:SW_Cherry_MX_PCB_1.25u -> Button_Switch_Keyboard:SW_Cherry_MX_1.25u_PCB
- SW62: footprint PCM_Switch_Keyboard_Cherry_MX:SW_Cherry_MX_PCB_6.50u -> Button_Switch_Keyboard:SW_Cherry_MX_6.25u_PCB
- moved R5 102.2 mm to (86.0, 76.2), turned to -90 degrees
- moved C1 85.7 mm to (122.9, 98.1)
- moved U2 83.0 mm to (264.2, 95.9), turned to -90 degrees
- moved R4 81.1 mm to (83.5, 76.2), turned to -90 degrees
- moved U1 79.6 mm to (130.8, 95.6)
- moved C2 73.4 mm to (256.2, 98.4)
- moved R3 63.0 mm to (81.0, 76.2), turned to -90 degrees
- moved J1 49.2 mm to (72.5, 87.6)
- moved D15 45.2 mm to (339.1, 65.7), turned to 0 degrees
- moved D44 45.2 mm to (339.1, 103.8), turned to 0 degrees
- moved D30 45.2 mm to (339.1, 84.8), turned to 0 degrees
- moved D57 45.2 mm to (320.1, 122.9), turned to 0 degrees
- moved D58 45.2 mm to (339.1, 122.9), turned to 0 degrees
- moved D63 45.2 mm to (243.9, 141.9), turned to 0 degrees
- moved D67 45.2 mm to (320.1, 141.9), turned to 0 degrees
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Routing:
- net /CS: track 284.5 -> 417.0 mm, vias 5 -> 6
- net ADDR3: track 306.9 -> 432.4 mm, vias 5 -> 8
- net ADDR2: track 305.0 -> 420.4 mm, vias 5 -> 7
- net ROW3: track 424.2 -> 534.9 mm, vias 4 -> 7
- net ADDR1: track 309.2 -> 413.0 mm
- net ADDR0: track 318.1 -> 410.8 mm, vias 5 -> 7
- net ROW2: track 442.8 -> 531.6 mm, vias 4 -> 8
- net ROW4: track 460.7 -> 392.7 mm, vias 5 -> 6
- net RAW_COL11: track 121.6 -> 57.9 mm, vias 2 -> 0
- net VCC: track 490.9 -> 431.8 mm, vias 8 -> 18
- net RAW_COL13: track 186.8 -> 127.8 mm
- net RAW_COL12: track 166.3 -> 110.2 mm
- net ROW1: track 457.7 -> 513.0 mm, vias 3 -> 4
- net RAW_COL14: track 198.6 -> 147.9 mm
- net RAW_COL8: track 103.6 -> 145.3 mm, vias 3 -> 2
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Other:
- board size 317.5 x 103.2 mm -> 313.1 x 103.5 mm
- board text added: "Keyboard2B A.K. 2024"
- board text removed: "Keyboard2 A.K. 2024"

Commit message: Add mini version
Parts:
- removed C3: 1u, Capacitor_SMD:C_0805_2012Metric_Pad1.18x1.45mm_HandSolder
- removed C4, C7: 100n, Capacitor_SMD:C_0805_2012Metric_Pad1.18x1.45mm_HandSolder
- removed C5, C6: 22p, Capacitor_SMD:C_0805_2012Metric_Pad1.18x1.45mm_HandSolder
- removed D15, D30, D44, D58, D68: D, Diode_SMD:D_MiniMELF
- removed J4: USB_B_Mini, Connector_USB:USB_Mini-B_Wuerth_65100516121_Horizontal
- removed J5: Conn_02x03_Odd_Even, Connector_PinHeader_2.54mm:PinHeader_2x03_P2.54mm_Vertical
- removed R1, R2, R3, R4, R5: 10K, Resistor_SMD:R_0805_2012Metric_Pad1.20x1.40mm_HandSolder
- removed REF** (x4): MountingHole_3.2mm_M3_Pad_Via, MountingHole:MountingHole_3.2mm_M3_Pad_Via
- removed SW15, SW30, SW44, SW58, SW68: SW_Push, Button_Switch_Keyboard:SW_Cherry_MX_1.00u_PCB
- removed U3: ATmega16U4-A, Package_QFP:TQFP-44_10x10mm_P0.8mm
- removed Y1: Crystal, Crystal:Crystal_HC49-4H_Vertical
- added H1: MountingHole, MountingHole:MountingHole_2.7mm_M2.5_Pad_Via, F.Cu at (50.8, 103.1)
- added H2: MountingHole, MountingHole:MountingHole_2.7mm_M2.5_Pad_Via, F.Cu at (67.8, 142.5)
- added H3: MountingHole, MountingHole:MountingHole_2.7mm_M2.5_Pad_Via, F.Cu at (148.8, 83.7)
- added H4: MountingHole, MountingHole:MountingHole_2.7mm_M2.5_Pad_Via, F.Cu at (163.2, 140.3)
- added H5: MountingHole, MountingHole:MountingHole_2.7mm_M2.5_Pad_Via, F.Cu at (244.1, 83.8)
- added H6: MountingHole, MountingHole:MountingHole_2.7mm_M2.5_Pad_Via, F.Cu at (258.4, 139.6)
- added H7: MountingHole, MountingHole:MountingHole_2.7mm_M2.5_Pad_Via, F.Cu at (303.4, 92.6)
- added H8: MountingHole, MountingHole:MountingHole_2.7mm_M2.5_Pad_Via, F.Cu at (310.6, 140.2)
- added R8: 10K, Resistor_SMD:R_0805_2012Metric_Pad1.20x1.40mm_HandSolder, B.Cu at (74.7, 79.0)
- added R9: 10K, Resistor_SMD:R_0805_2012Metric_Pad1.20x1.40mm_HandSolder, B.Cu at (77.2, 79.0)
- R10: value 4K7 -> 10K
- R11, R12: value 22R -> 10K
- moved R10 109.3 mm to (79.8, 79.0), turned to -90 degrees
- moved R11 83.9 mm to (82.3, 79.0)
- moved R12 80.4 mm to (84.8, 79.0), turned to -90 degrees
- moved D16 4.71 mm to (54.4, 87.6)
- moved D45 4.65 mm to (61.5, 125.7)
- moved D13 4.60 mm to (278.4, 68.6)
- moved D63 4.60 mm to (240.3, 144.8)
- moved D64 4.60 mm to (259.3, 144.8)
- moved D67 4.60 mm to (316.5, 144.8)
- moved D11 4.58 mm to (240.3, 68.6)
- moved D6 4.56 mm to (145.0, 68.6)
- moved D8 4.56 mm to (183.1, 68.6)
- moved D9 4.56 mm to (202.2, 68.6)
- moved D1 4.56 mm to (49.8, 68.6)
- moved D2 4.56 mm to (68.8, 68.6)
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Connections:
- R10 pad 2: /RST -> ROW2
- R11 pad 1: /D+ -> VCC
- R11 pad 2: Net-(U3-D+) -> ROW3
- R12 pad 1: Net-(U3-D-) -> VCC
- R12 pad 2: /D- -> ROW4
- U2 pad 9: RAW_COL14 -> unconnected-(U2-~{Y6}-Pad9)
Routing:
- net ROW3: track 534.9 -> 347.7 mm, vias 7 -> 5
- net ROW2: track 531.6 -> 347.2 mm, vias 8 -> 4
- net ROW1: track 513.0 -> 341.9 mm, vias 4 -> 2
- net ROW0: track 529.3 -> 371.3 mm, vias 5 -> 2
- net /D+: track 151.3 -> 0.00 mm, vias 2 -> 0
- net /D-: track 151.2 -> 0.00 mm, vias 2 -> 0
- net RAW_COL14: track 147.9 -> 0.00 mm, vias 2 -> 0
- net ADDR3: track 432.4 -> 289.5 mm, vias 8 -> 4
- net ADDR2: track 420.4 -> 280.6 mm, vias 7 -> 3
- net /CS: track 417.0 -> 283.2 mm, vias 6 -> 5
- net ADDR1: track 413.0 -> 281.6 mm, vias 6 -> 4
- net ADDR0: track 410.8 -> 280.2 mm, vias 7 -> 4
- net VCC: track 431.8 -> 309.1 mm, vias 18 -> 6
- net ROW4: track 392.7 -> 357.2 mm, vias 6 -> 4
- net MISO: track 26.4 -> 0.00 mm
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Other:
- board size 313.1 x 103.5 mm -> 281.2 x 97 mm
- board text added: "Keyboard2mini A.K. 2025"
- board text removed: "Keyboard2B A.K. 2024"
